Commit message: re-introduced fixed joint between `root` and `world` in dedicated Gazebo xacro file Re: https://github.com/Kinovarobotics/kinova-ros/pull/219#issuecomment-487654396

File: kinova_description/urdf/j2n4s300_standalone.xacro (robot description, xacro)
@@ -18,3 +18,4 @@
   <xacro:property name="robot_root" value="root" />
   <xacro:j2n4s300  base_parent="${robot_root}"/>
+  <xacro:gazebo_world_link />
 </robot>

File: kinova_description/urdf/j2n6s200_standalone.xacro (robot description, xacro)
@@ -18,3 +18,4 @@
   <xacro:property name="robot_root" value="root" />
   <xacro:j2n6s200  base_parent="${robot_root}"/>
+  <xacro:gazebo_world_link />
 </robot>

File: kinova_description/urdf/j2n6s300_standalone.xacro (robot description, xacro)
@@ -15,6 +15,8 @@
 	xmlns:xacro="http://ros.org/wiki/xacro" name="j2n6s300">
   <xacro:include filename="$(find kinova_description)/urdf/j2n6s300.xacro"/>
+  <xacro:include filename="$(find kinova_description)/urdf/j2n6s300.xacro"/>
   <link name="root"/>
   <xacro:property name="robot_root" value="root" />
   <xacro:j2n6s300  base_parent="${robot_root}"/>
+  <xacro:gazebo_world_link />
 </robot>

File: kinova_description/urdf/j2n7s300_standalone.xacro (robot description, xacro)
@@ -18,3 +18,4 @@
   <xacro:property name="robot_root" value="root" />
   <xacro:j2n7s300  base_parent="${robot_root}"/>
+  <xacro:gazebo_world_link />
 </robot>

File: kinova_description/urdf/j2s6s300_standalone.xacro (robot description, xacro)
@@ -18,3 +18,4 @@
   <xacro:property name="robot_root" value="root" />
   <xacro:j2s6s300  base_parent="${robot_root}"/>
+  <xacro:gazebo_world_link />
 </robot>

File: kinova_description/urdf/j2s7s300_standalone.xacro (robot description, xacro)
@@ -18,3 +18,4 @@
   <xacro:property name="robot_root" value="root" />
   <xacro:j2s7s300  base_parent="${robot_root}"/>
+  <xacro:gazebo_world_link />
 </robot>

File: kinova_description/urdf/m1n4s200_standalone.xacro (robot description, xacro)
@@ -18,3 +18,4 @@
   <xacro:property name="robot_root" value="root" />
   <xacro:m1n4s200  base_parent="${robot_root}"/>
+  <xacro:gazebo_world_link />
 </robot>

File: kinova_description/urdf/m1n6s200_standalone.xacro (robot description, xacro)
@@ -18,3 +18,4 @@
   <xacro:property name="robot_root" value="root" />
   <xacro:m1n6s200  base_parent="${robot_root}"/>
+  <xacro:gazebo_world_link />
 </robot>

File: kinova_description/urdf/m1n6s300_standalone.xacro (robot description, xacro)
@@ -18,3 +18,4 @@
   <xacro:property name="robot_root" value="root" />
   <xacro:m1n6s300  base_parent="${robot_root}"/>
+  <xacro:gazebo_world_link />
 </robot>

File: kinova_description/urdf/two_arm_robot_example_standalone.xacro (robot description, xacro)
@@ -15,18 +15,5 @@
 	xmlns:xacro="http://ros.org/wiki/xacro" name="j2s6a300">
   <xacro:include filename="$(find kinova_description)/urdf/j2n6s300.xacro"/>
-  <link name="root">
-    <visual>
-      <origin xyz="0 0 0" rpy="0 0 0" />
-      <geometry>
-        <box size = "0 0 0"/>
-      </geometry>
-    </visual>
-    <collision>
-      <origin xyz="0 0 0" rpy="0 0 0" />
-      <geometry>
-        <box size = "0 0 0"/>
-      </geometry>
-    </collision>
-  </link>
+  <link name="root" />
 	<link name="left_arm_mount">
   </link>
@@ -45,3 +32,4 @@
   <xacro:j2n6s300  base_parent="left_arm_mount" prefix="left"/>
 	<xacro:j2n6s300  base_parent="right_arm_mount" prefix="right"/>
+  <xacro:gazebo_world_link />
 </robot>
